Commit message: change to enu, fail in gazebo

File: robotx_description/urdf/robotx_base.urdf.xacro (robot description, xacro)
@@ -24,5 +24,5 @@
         <link name="${position}_bouy_link">
             <collision>
-                <origin xyz="0 0 0" rpy="0 ${PI/2} 0"/>
+                <origin xyz="0 0 0" rpy="${PI/2} 0 0"/>
                 <geometry>
                     <cylinder length="${bouy_length}" radius="${bouy_radius}"/>
@@ -30,5 +30,5 @@
             </collision>
             <visual>
-                <origin xyz="0 0 0" rpy="0 ${PI/2}  0"/>
+                <origin xyz="0 0 0" rpy="${PI/2} 0  0"/>
                 <geometry>
                     <cylinder length="${bouy_length}" radius="${bouy_radius}"/>
@@ -39,6 +39,6 @@
                 <mass value="${bouy_mass}"/>
                 <inertia
-                    ixx="${bouy_mass / 12.0 * (3*(bouy_radius*bouy_radius + bouy_i_radius*bouy_i_radius) + bouy_length*bouy_length)}" ixy="0.0" ixz="0.0"
-                    iyy="${bouy_mass / 12.0 * (3*(bouy_radius*bouy_radius + bouy_i_radius*bouy_i_radius) + bouy_length*bouy_length)}" iyz="0.0"
+                    iyy="${bouy_mass / 12.0 * (3*(bouy_radius*bouy_radius + bouy_i_radius*bouy_i_radius) + bouy_length*bouy_length)}" ixy="0.0" ixz="0.0"
+                    ixx="${bouy_mass / 12.0 * (3*(bouy_radius*bouy_radius + bouy_i_radius*bouy_i_radius) + bouy_length*bouy_length)}" iyz="0.0"
                     izz="${bouy_mass / 12.0 * 3*(bouy_radius*bouy_radius + bouy_i_radius*bouy_i_radius)}"/>
             </inertial>
@@ -46,5 +46,5 @@
     </xacro:macro>
     <!-- support bars -->
-    <xacro:macro name="bars" params="position1 position2 sign_x sign_y sign_roll" >
+    <xacro:macro name="bars" params="position1 position2 sign_x sign_y sign_roll sign_pitch" >
         <joint name="${position1}_${position2}_bar_joint" type="fixed">
         <parent link="shelf_link"/>
@@ -54,5 +54,5 @@
     <link name="${position1}_${position2}_bar_link">
         <collision>
-            <origin xyz="${sign_x*shelf_length/2} ${sign_y*shelf_width/2} 0" rpy="${sign_roll*PI/8} 0 0"/>
+            <origin xyz="${sign_x*shelf_width/2} ${sign_y*shelf_length/2} 0" rpy="${sign_roll*PI/8} ${sign_pitch*PI/8} 0"/>
             <geometry>
                 <cylinder length="${shelf_height}" radius="0.01"/>
@@ -60,5 +60,5 @@
         </collision>
         <visual>
-            <origin xyz="${sign_x*shelf_length/2} ${sign_y*shelf_width/2} 0" rpy="${sign_roll*PI/8} 0 0"/>
+            <origin xyz="${sign_x*shelf_width/2} ${sign_y*shelf_length/2} 0" rpy="${sign_roll*PI/8} ${sign_pitch*PI/8} 0"/>
             <geometry>
                 <cylinder length="${shelf_height}" radius="0.01"/>
@@ -72,5 +72,5 @@
             <origin xyz="0 0 0" rpy="0 0 0"/>
             <geometry>
-                <box size="${bouy_length} ${bouy_sep+2*bouy_radius} 0.01"/>
+                <box size="${bouy_sep+2*bouy_radius} ${bouy_length} 0.01"/>
             </geometry>
         </collision>
@@ -80,5 +80,5 @@
         <parent link="base_link"/>
         <child link="left_bouy_link"/>
-        <origin xyz="0 -${bouy_sep/2} ${bouy_radius}" rpy="0 0 0"/>
+        <origin xyz="-${bouy_sep/2} 0 ${bouy_radius}" rpy="0 0 0"/>
     </joint>
     <!-- left bouy Link -->
@@ -88,5 +88,5 @@
         <parent link="base_link"/>
         <child link="right_bouy_link"/>
-        <origin xyz="0 ${bouy_sep/2} ${bouy_radius}" rpy="0 0 0"/>
+        <origin xyz="${bouy_sep/2} 0 ${bouy_radius}" rpy="0 0 0"/>
     </joint>
     <!-- right bouy Link -->
@@ -103,5 +103,5 @@
             <origin xyz="0 0 0" rpy="0 0 0"/>
             <geometry>
-                <box size="${shelf_length} ${shelf_width} ${shelf_thickness}"/>
+                <box size="${shelf_width} ${shelf_length} ${shelf_thickness}"/>
             </geometry>
         </collision>
@@ -109,5 +109,5 @@
             <origin xyz="0 0 0" rpy="0 0 0"/>
             <geometry>
-                <box size="${shelf_length} ${shelf_width} ${shelf_thickness}"/>
+                <box size="${shelf_width} ${shelf_length} ${shelf_thickness}"/>
             </geometry>
             <material name="yellow"/>
@@ -117,26 +117,26 @@
             <mass value="${shelf_mass}"/>
             <inertia
-                ixx="${shelf_mass / 12.0 * (shelf_length*shelf_length + shelf_thickness*shelf_thickness)}" ixy="0.0" ixz="0.0"
-                iyy="${shelf_mass / 12.0 * (shelf_length*shelf_length + shelf_width*shelf_width)}" iyz="0.0"
+                iyy="${shelf_mass / 12.0 * (shelf_length*shelf_length + shelf_thickness*shelf_thickness)}" ixy="0.0" ixz="0.0"
+                ixx="${shelf_mass / 12.0 * (shelf_length*shelf_length + shelf_width*shelf_width)}" iyz="0.0"
                 izz="${shelf_mass / 12.0 * (shelf_width*shelf_width + shelf_thickness*shelf_thickness)}"/>
         </inertial>
     </link>
     <!-- bars -->
-    <xacro:bars position1="front" position2="left" sign_x="1" sign_y="-1" sign_roll="-1"/>
-    <xacro:bars position1="front" position2="right" sign_x="1" sign_y="1" sign_roll="1"/>
-    <xacro:bars position1="rear" position2="left" sign_x="-1" sign_y="-1" sign_roll="-1"/>
-    <xacro:bars position1="rear" position2="right" sign_x="-1" sign_y="1" sign_roll="1"/>
+    <xacro:bars position1="front" position2="left" sign_x="-1" sign_y="1" sign_roll="1" sign_pitch="1"/>
+    <xacro:bars position1="front" position2="right" sign_x="1" sign_y="1" sign_roll="1" sign_pitch="-1"/>
+    <xacro:bars position1="rear" position2="left" sign_x="-1" sign_y="-1" sign_roll="-1" sign_pitch="1"/>
+    <xacro:bars position1="rear" position2="right" sign_x="1" sign_y="-1" sign_roll="-1" sign_pitch="-1"/>
     <!-- sensor box joint-->
-    <joint name="sensor_box_joint" type="fixed">
+    <joint name="imu_joint" type="fixed">
         <parent link="shelf_link"/>
-        <child link="sensor_box_link"/>
-        <origin xyz="0.5 0 ${sensor_box_thickness/2+shelf_thickness/2}" rpy="0 0 0"/>
+        <child link="base_imu_link"/>
+        <origin xyz="0 0.5 ${sensor_box_thickness/2+shelf_thickness/2}" rpy="0 0 0"/>
     </joint>
     <!-- sensor box -->
-    <link name="sensor_box_link">
+    <link name="base_imu_link">
         <collision>
             <origin xyz="0 0 0" rpy="0 0 0"/>
             <geometry>
-                <box size="${sensor_box_length} ${sensor_box_width} ${sensor_box_thickness}"/>
+                <box size="${sensor_box_width} ${sensor_box_length} ${sensor_box_thickness}"/>
             </geometry>
         </collision>
@@ -144,5 +144,5 @@
             <origin xyz="0 0 0" rpy="0 0 0"/>
             <geometry>
-                <box size="${sensor_box_length} ${sensor_box_width} ${sensor_box_thickness}"/>
+                <box size="${sensor_box_width} ${sensor_box_length} ${sensor_box_thickness}"/>
             </geometry>
             <material name="blue"/>
@@ -152,6 +152,6 @@
             <mass value="${sensor_box_mass}"/>
             <inertia
-                ixx="${sensor_box_mass / 12.0 * (sensor_box_length*sensor_box_length + sensor_box_thickness*sensor_box_thickness)}" ixy="0.0" ixz="0.0"
-                iyy="${sensor_box_mass / 12.0 * (sensor_box_length*sensor_box_length + sensor_box_width*sensor_box_width)}" iyz="0.0"
+                iyy="${sensor_box_mass / 12.0 * (sensor_box_length*sensor_box_length + sensor_box_thickness*sensor_box_thickness)}" ixy="0.0" ixz="0.0"
+                ixx="${sensor_box_mass / 12.0 * (sensor_box_length*sensor_box_length + sensor_box_width*sensor_box_width)}" iyz="0.0"
                 izz="${sensor_box_mass / 12.0 * (sensor_box_width*sensor_box_width + sensor_box_thickness*sensor_box_thickness)}"/>
         </inertial>

File: robotx_description/urdf/sensor.urdf.xacro (robot description, xacro)
@@ -8,20 +8,53 @@
     <xacro:property name="camera_height" value="0.1" />
     <!-- camera array joint -->
-    <xacro:macro name="spot_camera_array" params="position1">
-        <joint name="${position1}_camera_array_joint" type="fixed">
-            <origin xyz="0 0 0" rpy="0 0 0" />
-            <parent link="shelf_link"/>
-            <child link="${position1}_stereo/camera_link"/>
-        </joint>
-        <link name="${position1}_stereo/camera_link"/>
+    <xacro:macro name="spot_camera" params="position1 x y z yaw">
+        <joint name="${position1}_camera_joint" type="fixed">
+            <origin xyz="${y} ${x} ${z}" rpy="0 0 ${yaw}" />
+            <parent link="shelf_link"/>
+            <child link="${position1}/camera_link"/>
+        </joint>
+        <link name="${position1}/camera_link">
+            <visual>
+                <origin xyz="0 0 0" rpy="0 0 0" />
+                <geometry>
+                    <mesh filename="package://hector_sensors_description/meshes/thermaleye_camera/thermaleye_camera_hector_v2.dae"/>
+                </geometry>
+            </visual>
+            <collision>
+                <origin xyz="0 0 0" rpy="0 0 0" />
+                <geometry>
+                    <mesh filename="package://hector_sensors_description/meshes/thermaleye_camera/thermaleye_camera_hector_v2.stl"/>
+                </geometry>
+            </collision>
+        </link>
     </xacro:macro>
-    <!-- Set up camera linkage and configuration -->
-    <xacro:macro name="spot_camera" params="position1 position2 x y z yaw">
+    <xacro:macro name="underwater_camera" params="position1 x y z roll yaw">
+        <joint name="${position1}_camera_joint" type="fixed">
+            <origin xyz="${y} ${x} ${z}" rpy="0 ${roll} ${yaw}" />
+            <parent link="shelf_link"/>
+            <child link="${position1}/camera_link"/>
+        </joint>
+        <link name="${position1}/camera_link">
+            <visual>
+                <origin xyz="0 0 0" rpy="0 0 0" />
+                <geometry>
+                    <mesh filename="package://hector_sensors_description/meshes/thermaleye_camera/thermaleye_camera_hector_v2.dae"/>
+                </geometry>
+            </visual>
+            <collision>
+                <origin xyz="0 0 0" rpy="0 0 0" />
+                <geometry>
+                    <mesh filename="package://hector_sensors_description/meshes/thermaleye_camera/thermaleye_camera_hector_v2.stl"/>
+                </geometry>
+            </collision>
+        </link>
+    </xacro:macro>
+    <xacro:macro name="stereo_camera" params="position1 position2 x y z roll yaw">
         <joint name="${position1}_${position2}_camera_joint" type="fixed">
-            <origin xyz="${x} ${y} ${z+shelf_thickness/2}" rpy="0 0 ${yaw}" />
-            <parent link="${position1}_stereo/camera_link"/>
-            <child link="${position1}_stereo/${position2}/camera_link" />
-        </joint>
-        <link name="${position1}_stereo/${position2}/camera_link">
+            <origin xyz="${y} ${x} ${z}" rpy="0 ${roll} ${yaw}" />
+            <parent link="shelf_link"/>
+            <child link="${position1}/${position2}/camera_link"/>
+        </joint>
+        <link name="${position1}/${position2}/camera_link">
             <visual>
                 <origin xyz="0 0 0" rpy="0 0 0" />
@@ -37,14 +70,4 @@
             </collision>
         </link>
-    </xacro:macro>
-    <xacro:macro name="imu" params="position1 position2 x y">
-        <joint name="${position1}_${position2}_imu_joint" type="fixed">
-            <origin xyz="0 0 ${shelf_thickness/2}" rpy="0 0 0" />
-            <parent link="imu_array_link"/>
-            <!--child link="${position1}_${position2}_imu_link"/-->
-            <child link="base_imu_link"/>
-        </joint>
-        <!--link name="${position1}_${position2}_imu_link"/-->
-        <link name="base_imu_link"/>
     </xacro:macro>
     <joint name="gps_joint" type="fixed">
@@ -68,24 +91,10 @@
         </collision>
     </link>
-    <joint name="imu_array_joint" type="fixed">
-        <origin xyz="0 0 0" rpy="0 0 0" />
-        <parent link="shelf_link"/>
-        <child link="imu_array_link"/>
-    </joint>
-    <link name="imu_array_link" />
-    <xacro:imu position1="middle" position2="middle" x="0" y="0" />
-    <!--xacro:imu position1="front" position2="left" x="${shelf_length/2}" y="-${shelf_width/2}" />
-    <xacro:imu position1="front" position2="right" x="${shelf_length/2}" y="-${shelf_width/2}" />
-    <xacro:imu position1="rear" position2="left" x="${shelf_length/2}" y="-${shelf_width/2}" />
-    <xacro:imu position1="rear" position2="right" x="${shelf_length/2}" y="-${shelf_width/2}" /-->
-    <xacro:spot_camera_array position1="bow" />
-    <xacro:spot_camera_array position1="port" />
-    <xacro:spot_camera_array position1="starboard" />
-    <xacro:spot_camera position1="bow" position2="left" x="${shelf_length/2}" y="-${shelf_width/2}" z="${5*camera_height}" yaw="0"/>
-    <xacro:spot_camera position1="bow" position2="right" x="${shelf_length/2}" y="${shelf_width/2}" z="${5*camera_height}" yaw="0"/>
-    <xacro:spot_camera position1="port" position2="left" x="-${shelf_length/2}" y="-${shelf_width/2}" z="${camera_height}" yaw="-${PI/2}"/>
-    <xacro:spot_camera position1="port" position2="right" x="${shelf_length/2}" y="-${shelf_width/2}" z="${camera_height}" yaw="-${PI/2}"/>
-    <xacro:spot_camera position1="starboard" position2="left" x="${shelf_length/2}" y="${shelf_width/2}" z="${camera_height}" yaw="${PI/2}"/>
-    <xacro:spot_camera position1="starboard" position2="right" x="-${shelf_length/2}" y="${shelf_width/2}" z="${camera_height}" yaw="${PI/2}"/>
+    <xacro:stereo_camera position1="bow" position2="left" x="${shelf_length/2+0.2}" y="-${shelf_width/4}" z="${camera_height}" roll="0.157" yaw="${PI/2}"/>
+    <xacro:stereo_camera position1="bow" position2="right" x="${shelf_length/2+0.2}" y="${shelf_width/4}" z="${camera_height}" roll="0.157" yaw="${PI/2}"/>
+    <xacro:underwater_camera position1="underwater" x="${shelf_length/2}" y="${shelf_width/2}" z="-1" roll="${PI/2}" yaw="-${PI/2}"/>
+    <xacro:spot_camera position1="port" x="${shelf_length/2}" y="-${shelf_width/2}" z="${camera_height}" yaw="-${PI}"/>
+    <xacro:spot_camera position1="starboard" x="${shelf_length/2}" y="${shelf_width/2}" z="${camera_height}" yaw="0"/>
+    <xacro:spot_camera position1="transom" x="-${1.8*shelf_width/2}" y="0" z="${camera_height}" yaw="-${PI/2}"/>
     <!--kinect camera >
     <joint name="kinect_camera_joint" type="fixed">
@@ -169,5 +178,5 @@
     <xacro:if value="$(arg lidar_enabled)">
         <joint name="hokuyo_joint" type="fixed">
-            <origin xyz="${shelf_length/2} 0.0 0.4" rpy="0 0 0"/>
+            <origin xyz="0 ${shelf_length/2} 0.4" rpy="0 0 ${PI/2}"/>
             <parent link="shelf_link"/>
             <child link="hokuyo_link"/>
