Commit message: add lidar

File: robotx_description/urdf/sensor.urdf.xacro (robot description, xacro)
@@ -8,5 +8,5 @@
     <xacro:property name="camera_height" value="0.1" />
     <!-- camera array joint -->
-    <xacro:macro name="sport_camera_array" params="position1">
+    <xacro:macro name="spot_camera_array" params="position1">
         <joint name="${position1}_camera_array_joint" type="fixed">
             <origin xyz="0 0 0" rpy="0 0 0" />
@@ -77,7 +77,7 @@
     <xacro:imu position1="rear" position2="left" x="${shelf_length/2}" y="-${shelf_width/2}" />
     <xacro:imu position1="rear" position2="right" x="${shelf_length/2}" y="-${shelf_width/2}" /-->
-    <xacro:sport_camera_array position1="bow" />
-    <xacro:sport_camera_array position1="port" />
-    <xacro:sport_camera_array position1="starboard" />
+    <xacro:spot_camera_array position1="bow" />
+    <xacro:spot_camera_array position1="port" />
+    <xacro:spot_camera_array position1="starboard" />
     <xacro:spot_camera position1="bow" position2="left" x="${shelf_length/2}" y="-${shelf_width/2}" z="${5*camera_height}" yaw="0"/>
     <xacro:spot_camera position1="bow" position2="right" x="${shelf_length/2}" y="${shelf_width/2}" z="${5*camera_height}" yaw="0"/>
@@ -164,9 +164,9 @@
         </link>
     </xacro:if -->
-    <!-- Hokuyo Laser >
+    <!-- Hokuyo Laser -->
     <xacro:if value="$(arg lidar_enabled)">
         <joint name="hokuyo_joint" type="fixed">
-            <origin xyz="0.2 0.0 0.2" rpy="0 0 0"/>
-            <parent link="base_link"/>
+            <origin xyz="${shelf_length/2} 0.0 0.4" rpy="0 0 0"/>
+            <parent link="shelf_link"/>
             <child link="hokuyo_link"/>
         </joint>
@@ -190,4 +190,4 @@
             </inertial>
         </link>
-    </xacro:if-->
+    </xacro:if>
 </robot>

Commit message: ground_truth

File: robotx_description/urdf/sensor.urdf.xacro (robot description, xacro)
@@ -167,5 +167,5 @@
     <xacro:if value="$(arg lidar_enabled)">
         <joint name="hokuyo_joint" type="fixed">
-            <origin xyz="${shelf_length/2} 0.0 0.4" rpy="0 0 0"/>
+            <origin xyz="${shelf_length/2} 0.0 -0.5" rpy="0 0 0"/>
             <parent link="shelf_link"/>
             <child link="hokuyo_link"/>

Commit message: land test 20161114

File: robotx_description/urdf/sensor.urdf.xacro (robot description, xacro)
@@ -42,7 +42,9 @@
             <origin xyz="0 0 ${shelf_thickness/2}" rpy="0 0 0" />
             <parent link="imu_array_link"/>
-            <child link="${position1}_${position2}_imu_link"/>
+            <!--child link="${position1}_${position2}_imu_link"/-->
+            <child link="base_imu_link"/>
         </joint>
-        <link name="${position1}_${position2}_imu_link"/>
+        <!--link name="${position1}_${position2}_imu_link"/-->
+        <link name="base_imu_link"/>
     </xacro:macro>
     <joint name="gps_joint" type="fixed">

Commit message: gazebo to sim wamv's r l

File: robotx_description/urdf/sensor.urdf.xacro (robot description, xacro)
@@ -178,5 +178,5 @@
     <xacro:if value="$(arg lidar_enabled)">
         <joint name="hokuyo_joint" type="fixed">
-            <origin xyz="${shelf_length/2} 0 0.4" rpy="0 0.157 0"/>
+            <origin xyz="${shelf_length/2} 0 0.4" rpy="0 0 0"/>
             <parent link="shelf_link"/>
             <child link="hokuyo_link"/>

Commit message: urdf change to camera coordinates

File: robotx_description/urdf/sensor.urdf.xacro (robot description, xacro)
@@ -10,5 +10,5 @@
     <xacro:macro name="spot_camera" params="position1 x y z yaw">
         <joint name="${position1}_camera_joint" type="fixed">
-            <origin xyz="${x} ${y} ${z}" rpy="0 0 ${yaw}" />
+				<origin xyz="${x} ${y} ${z}" rpy="-${PI/2} 0 ${-1*PI/2-yaw}" />
             <parent link="shelf_link"/>
             <child link="${position1}/camera_link"/>
@@ -16,5 +16,5 @@
         <link name="${position1}/camera_link">
             <visual>
-                <origin xyz="0 0 0" rpy="0 0 0" />
+					<origin xyz="0 0 0" rpy="0 -${PI/2} 0" />
                 <geometry>
                     <mesh filename="package://hector_sensors_description/meshes/thermaleye_camera/thermaleye_camera_hector_v2.dae"/>
@@ -22,5 +22,5 @@
             </visual>
             <collision>
-                <origin xyz="0 0 0" rpy="0 0 0" />
+					<origin xyz="0 0 0" rpy="0 -${PI/2} 0" />
                 <geometry>
                     <mesh filename="package://hector_sensors_description/meshes/thermaleye_camera/thermaleye_camera_hector_v2.stl"/>
@@ -29,7 +29,7 @@
         </link>
     </xacro:macro>
-    <xacro:macro name="underwater_camera" params="position1 x y z roll yaw">
+    <xacro:macro name="underwater_camera" params="position1 x y z">
         <joint name="${position1}_camera_joint" type="fixed">
-            <origin xyz="${x} ${y} ${z}" rpy="0 ${roll} ${yaw}" />
+				<origin xyz="${x} ${y} ${z}" rpy="0 ${PI} ${PI/2} " />
             <parent link="shelf_link"/>
             <child link="${position1}/camera_link"/>
@@ -37,5 +37,5 @@
         <link name="${position1}/camera_link">
             <visual>
-                <origin xyz="0 0 0" rpy="0 0 0" />
+					<origin xyz="0 0 0" rpy="0 -${PI/2} 0" />
                 <geometry>
                     <mesh filename="package://hector_sensors_description/meshes/thermaleye_camera/thermaleye_camera_hector_v2.dae"/>
@@ -43,5 +43,5 @@
             </visual>
             <collision>
-                <origin xyz="0 0 0" rpy="0 0 0" />
+					<origin xyz="0 0 0" rpy="0 -${PI/2} 0" />
                 <geometry>
                     <mesh filename="package://hector_sensors_description/meshes/thermaleye_camera/thermaleye_camera_hector_v2.stl"/>
@@ -50,7 +50,7 @@
         </link>
     </xacro:macro>
-    <xacro:macro name="stereo_camera" params="position1 position2 x y z roll yaw">
+    <xacro:macro name="stereo_camera" params="position1 position2 x y z pitch">
         <joint name="${position1}_${position2}_camera_joint" type="fixed">
-            <origin xyz="${x} ${y} ${z}" rpy="0 ${roll} ${yaw}" />
+				<origin xyz="${x} ${y} ${z}" rpy="${-PI/2-pitch} 0 ${-PI/2}" />
             <parent link="shelf_link"/>
             <child link="${position1}/${position2}/camera_link"/>
@@ -58,5 +58,5 @@
         <link name="${position1}/${position2}/camera_link">
             <visual>
-                <origin xyz="0 0 0" rpy="0 0 0" />
+					<origin xyz="0 0 0" rpy="0 ${-1*PI/2} 0" />
                 <geometry>
                     <mesh filename="package://hector_sensors_description/meshes/thermaleye_camera/thermaleye_camera_hector_v2.dae"/>
@@ -64,5 +64,5 @@
             </visual>
             <collision>
-                <origin xyz="0 0 0" rpy="0 0 0" />
+					<origin xyz="0 0 0" rpy="0 ${-1*PI/2} 0" />
                 <geometry>
                     <mesh filename="package://hector_sensors_description/meshes/thermaleye_camera/thermaleye_camera_hector_v2.stl"/>
@@ -91,10 +91,10 @@
         </collision>
     </link>
-    <xacro:stereo_camera position1="bow" position2="left" x="${shelf_length/2+0.2}" y="${shelf_width/4}" z="${camera_height}" roll="0.157" yaw="0"/>
-    <xacro:stereo_camera position1="bow" position2="right" x="${shelf_length/2+0.2}" y="-${shelf_width/4}" z="${camera_height}" roll="0.157" yaw="0"/>
-    <xacro:underwater_camera position1="underwater" x="${shelf_length/2}" y="${shelf_width/2}" z="-1" roll="${PI/2}" yaw="0"/>
-    <xacro:spot_camera position1="port" x="${shelf_length/2}" y="${shelf_width/2}" z="${camera_height}" yaw="${PI/2}"/>
-    <xacro:spot_camera position1="starboard" x="${shelf_length/2}" y="-${shelf_width/2}" z="${camera_height}" yaw="-${PI/2}"/>
-    <xacro:spot_camera position1="transom" x="-${1.8*shelf_width/2}" y="0" z="${camera_height}" yaw="${PI}"/>
+    <xacro:stereo_camera position1="bow" position2="left" x="${shelf_length/2+0.2}" y="${shelf_width/4}" z="${camera_height}" pitch="0.157" />
+    <xacro:stereo_camera position1="bow" position2="right" x="${shelf_length/2+0.2}" y="-${shelf_width/4}" z="${camera_height}" pitch="0.157" />
+    <xacro:underwater_camera position1="underwater" x="${shelf_length/2}" y="${shelf_width/2}" z="-1" />
+    <xacro:spot_camera position1="port" x="${shelf_length/2}" y="${shelf_width/2}" z="${camera_height}" yaw="-${PI/2}"/>
+    <xacro:spot_camera position1="starboard" x="${shelf_length/2}" y="-${shelf_width/2}" z="${camera_height}" yaw="${PI/2}"/>
+    <xacro:spot_camera position1="transom" x="-${1.8*shelf_width/2}" y="0" z="${camera_height}" yaw="-${PI}"/>
     <!--kinect camera >
     <joint name="kinect_camera_joint" type="fixed">

Commit message: revert back camera due to image is on x_optic

File: robotx_description/urdf/sensor.urdf.xacro (robot description, xacro)
@@ -10,5 +10,5 @@
     <xacro:macro name="spot_camera" params="position1 x y z yaw">
         <joint name="${position1}_camera_joint" type="fixed">
-				<origin xyz="${x} ${y} ${z}" rpy="-${PI/2} 0 ${-1*PI/2-yaw}" />
+            <origin xyz="${x} ${y} ${z}" rpy="0 0 ${yaw}" />
             <parent link="shelf_link"/>
             <child link="${position1}/camera_link"/>
@@ -16,5 +16,5 @@
         <link name="${position1}/camera_link">
             <visual>
-					<origin xyz="0 0 0" rpy="0 -${PI/2} 0" />
+                <origin xyz="0 0 0" rpy="0 0 0" />
                 <geometry>
                     <mesh filename="package://hector_sensors_description/meshes/thermaleye_camera/thermaleye_camera_hector_v2.dae"/>
@@ -22,5 +22,5 @@
             </visual>
             <collision>
-					<origin xyz="0 0 0" rpy="0 -${PI/2} 0" />
+                <origin xyz="0 0 0" rpy="0 0 0" />
                 <geometry>
                     <mesh filename="package://hector_sensors_description/meshes/thermaleye_camera/thermaleye_camera_hector_v2.stl"/>
@@ -29,7 +29,7 @@
         </link>
     </xacro:macro>
-    <xacro:macro name="underwater_camera" params="position1 x y z">
+    <xacro:macro name="underwater_camera" params="position1 x y z roll yaw">
         <joint name="${position1}_camera_joint" type="fixed">
-				<origin xyz="${x} ${y} ${z}" rpy="0 ${PI} ${PI/2} " />
+            <origin xyz="${x} ${y} ${z}" rpy="0 ${roll} ${yaw}" />
             <parent link="shelf_link"/>
             <child link="${position1}/camera_link"/>
@@ -37,5 +37,5 @@
         <link name="${position1}/camera_link">
             <visual>
-					<origin xyz="0 0 0" rpy="0 -${PI/2} 0" />
+                <origin xyz="0 0 0" rpy="0 0 0" />
                 <geometry>
                     <mesh filename="package://hector_sensors_description/meshes/thermaleye_camera/thermaleye_camera_hector_v2.dae"/>
@@ -43,5 +43,5 @@
             </visual>
             <collision>
-					<origin xyz="0 0 0" rpy="0 -${PI/2} 0" />
+                <origin xyz="0 0 0" rpy="0 0 0" />
                 <geometry>
                     <mesh filename="package://hector_sensors_description/meshes/thermaleye_camera/thermaleye_camera_hector_v2.stl"/>
@@ -50,7 +50,7 @@
         </link>
     </xacro:macro>
-    <xacro:macro name="stereo_camera" params="position1 position2 x y z pitch">
+    <xacro:macro name="stereo_camera" params="position1 position2 x y z roll yaw">
         <joint name="${position1}_${position2}_camera_joint" type="fixed">
-				<origin xyz="${x} ${y} ${z}" rpy="${-PI/2-pitch} 0 ${-PI/2}" />
+            <origin xyz="${x} ${y} ${z}" rpy="0 ${roll} ${yaw}" />
             <parent link="shelf_link"/>
             <child link="${position1}/${position2}/camera_link"/>
@@ -58,5 +58,5 @@
         <link name="${position1}/${position2}/camera_link">
             <visual>
-					<origin xyz="0 0 0" rpy="0 ${-1*PI/2} 0" />
+                <origin xyz="0 0 0" rpy="0 0 0" />
                 <geometry>
                     <mesh filename="package://hector_sensors_description/meshes/thermaleye_camera/thermaleye_camera_hector_v2.dae"/>
@@ -64,5 +64,5 @@
             </visual>
             <collision>
-					<origin xyz="0 0 0" rpy="0 ${-1*PI/2} 0" />
+                <origin xyz="0 0 0" rpy="0 0 0" />
                 <geometry>
                     <mesh filename="package://hector_sensors_description/meshes/thermaleye_camera/thermaleye_camera_hector_v2.stl"/>
@@ -91,10 +91,10 @@
         </collision>
     </link>
-    <xacro:stereo_camera position1="bow" position2="left" x="${shelf_length/2+0.2}" y="${shelf_width/4}" z="${camera_height}" pitch="0.157" />
-    <xacro:stereo_camera position1="bow" position2="right" x="${shelf_length/2+0.2}" y="-${shelf_width/4}" z="${camera_height}" pitch="0.157" />
-    <xacro:underwater_camera position1="underwater" x="${shelf_length/2}" y="${shelf_width/2}" z="-1" />
-    <xacro:spot_camera position1="port" x="${shelf_length/2}" y="${shelf_width/2}" z="${camera_height}" yaw="-${PI/2}"/>
-    <xacro:spot_camera position1="starboard" x="${shelf_length/2}" y="-${shelf_width/2}" z="${camera_height}" yaw="${PI/2}"/>
-    <xacro:spot_camera position1="transom" x="-${1.8*shelf_width/2}" y="0" z="${camera_height}" yaw="-${PI}"/>
+    <xacro:stereo_camera position1="bow" position2="left" x="${shelf_length/2+0.2}" y="${shelf_width/4}" z="${camera_height}" roll="0.157" yaw="0"/>
+    <xacro:stereo_camera position1="bow" position2="right" x="${shelf_length/2+0.2}" y="-${shelf_width/4}" z="${camera_height}" roll="0.157" yaw="0"/>
+    <xacro:underwater_camera position1="underwater" x="${shelf_length/2}" y="${shelf_width/2}" z="-1" roll="${PI/2}" yaw="0"/>
+    <xacro:spot_camera position1="port" x="${shelf_length/2}" y="${shelf_width/2}" z="${camera_height}" yaw="${PI/2}"/>
+    <xacro:spot_camera position1="starboard" x="${shelf_length/2}" y="-${shelf_width/2}" z="${camera_height}" yaw="-${PI/2}"/>
+    <xacro:spot_camera position1="transom" x="-${1.8*shelf_width/2}" y="0" z="${camera_height}" yaw="${PI}"/>
     <!--kinect camera >
     <joint name="kinect_camera_joint" type="fixed">
