Commit message: add zed depth cam/use kinect gazebo

File: robotx_description/urdf/sensor.urdf.xacro (robot description, xacro)
@@ -2,205 +2,222 @@
 <!-- modified by ren ye on 2016-07-22 -->
 <robot name="robotx_sensors" xmlns:xacro="http://ros.org/wiki/xacro" >
-		<xacro:property name="M_PI" value="3.1415926535897931" />
-		<xacro:property name="shelf_length" value="1.85" />
-		<xacro:property name="shelf_width" value="1.01" />
-		<xacro:property name="shelf_thickness" value="0.1" />
-		<xacro:property name="camera_height" value="0.1" />
-		<!-- camera array joint -->
-		<xacro:macro name="spot_camera" params="position1 x y z yaw">
-				<joint name="${position1}_camera_joint" type="fixed">
-						<origin xyz="${x} ${y} ${z}" rpy="0 0 ${yaw}" />
-						<parent link="shelf_link"/>
-						<child link="${position1}/camera_link"/>
-				</joint>
-				<link name="${position1}/camera_link">
-						<visual>
-								<origin xyz="0 0 0" rpy="0 0 0" />
-								<geometry>
-										<mesh filename="package://hector_sensors_description/meshes/thermaleye_camera/thermaleye_camera_hector_v2.dae" />
-								</geometry>
-						</visual>
-						<collision>
-								<origin xyz="0 0 0" rpy="0 0 0" />
-								<geometry>
-										<mesh filename="package://hector_sensors_description/meshes/thermaleye_camera/thermaleye_camera_hector_v2.stl"/>
-								</geometry>
-						</collision>
-				</link>
-		</xacro:macro>
-		<xacro:macro name="underwater_camera" params="position1 x y z roll yaw">
-				<joint name="${position1}_camera_joint" type="fixed">
-						<origin xyz="${x} ${y} ${z}" rpy="0 ${roll} ${yaw}" />
-						<parent link="shelf_link"/>
-						<child link="${position1}/camera_link"/>
-				</joint>
-				<link name="${position1}/camera_link">
-						<visual>
-								<origin xyz="0 0 0" rpy="0 0 0" />
-								<geometry>
-										<mesh filename="package://hector_sensors_description/meshes/thermaleye_camera/thermaleye_camera_hector_v2.dae"/>
-								</geometry>
-						</visual>
-						<collision>
-								<origin xyz="0 0 0" rpy="0 0 0" />
-								<geometry>
-										<mesh filename="package://hector_sensors_description/meshes/thermaleye_camera/thermaleye_camera_hector_v2.stl"/>
-								</geometry>
-						</collision>
-				</link>
-		</xacro:macro>
-		<xacro:macro name="stereo_camera" params="position1 position2 x y z roll yaw">
-				<joint name="${position1}_${position2}_camera_joint" type="fixed">
-						<origin xyz="${x} ${y} ${z}" rpy="0 ${roll} ${yaw}" />
-						<parent link="shelf_link"/>
-						<child link="${position1}/${position2}/camera_link"/>
-				</joint>
-				<link name="${position1}/${position2}/camera_link">
-						<visual>
-								<origin xyz="0 0 0" rpy="0 0 0" />
-								<geometry>
-										<mesh filename="package://hector_sensors_description/meshes/thermaleye_camera/thermaleye_camera_hector_v2.dae"/>
-								</geometry>
-						</visual>
-						<collision>
-								<origin xyz="0 0 0" rpy="0 0 0" />
-								<geometry>
-										<mesh filename="package://hector_sensors_description/meshes/thermaleye_camera/thermaleye_camera_hector_v2.stl"/>
-								</geometry>
-						</collision>
-				</link>
-		</xacro:macro>
-		<joint name="gps_joint" type="fixed">
-				<origin xyz="0 0 ${shelf_thickness*6}" rpy="0 0 0" />
-				<parent link="shelf_link"/>
-				<child link="gps_link"/>
-		</joint>
-		<link name="gps_link">
-				<visual>
-						<origin xyz="0 0 0" rpy="0 0 0"/>
-						<geometry>
-								<cylinder length="0.08" radius="0.1" />
-						</geometry>
-						<material name="white" />
-				</visual>
-				<collision>
-						<origin xyz="0 0 0" rpy="0 0 0"/>
-						<geometry>
-								<cylinder length="0.08" radius="0.1" />
-						</geometry>
-				</collision>
-		</link>
-		<xacro:unless value="$(arg zed_enabled)" >
-		<xacro:stereo_camera position1="bow" position2="left" x="${shelf_length/2+0.2}" y="${shelf_width/4}" z="${camera_height}" roll="0.157" yaw="0"/>
-		<xacro:stereo_camera position1="bow" position2="right" x="${shelf_length/2+0.2}" y="-${shelf_width/4}" z="${camera_height}" roll="0.157" yaw="0"/>
-		</xacro:unless>
-		<xacro:underwater_camera position1="underwater" x="${shelf_length/2}" y="${shelf_width/2}" z="-1" roll="${PI/2}" yaw="0"/>
-		<xacro:spot_camera position1="port" x="${shelf_length/2}" y="${shelf_width/2}" z="${camera_height}" yaw="${PI/2}"/>
-		<xacro:spot_camera position1="starboard" x="${shelf_length/2}" y="-${shelf_width/2}" z="${camera_height}" yaw="-${PI/2}"/>
-		<xacro:spot_camera position1="transom" x="-${1.8*shelf_width/2}" y="0" z="${camera_height}" yaw="${PI}"/>
-		<!--zed camera -->
-		<xacro:if value="$(arg zed_enabled)" >
-				<joint name="zed_camera_joint" type="fixed">
-						<origin xyz="${shelf_length/2+0.2} 0 ${camera_height}" rpy="0 0 0" />
-						<parent link="shelf_link"/>
-						<child link="bow/camera_link"/>
-				</joint>
-				<link name="bow/camera_link">
-						<inertial>
-								<mass value="0.01" />
-								<origin xyz="0 0 0" rpy="0 0 0"/>
-								<inertia ixx="2.632e-4" ixy="0" ixz="0" iyy="2.632e-4" iyz="0" izz="1.62e-4" />
-						</inertial>
-						<visual>
-								<origin xyz="0 0 0" rpy="${PI/2} 0 ${PI/2}" />
-								<geometry>
-										<mesh filename="package://robotx_description/meshes/zed_model.dae" scale="0.05 0.05 0.05"/>
-								</geometry>
-						</visual>
-						<collision>
-								<origin xyz="0 0 0" rpy="0 0 0" />
-								<geometry>
-										<mesh filename="package://robotx_description/meshes/zed_model.dae" scale="0.05 0.05 0.05"/>
-								</geometry>
-						</collision>
-				</link>
-				<joint name="zed_camera_depth_joint" type="fixed">
-						<origin xyz="0.0 0.0 0.0" rpy="0 0 0" />
-						<parent link="bow/camera_link" />
-						<child link="zed_camera_depth_frame"/>
-				</joint>
-				<link name="zed_camera_depth_frame"/>
-				<joint name="zed_camera_depth_optical_joint" type="fixed">
-						<origin xyz="0 0 0" rpy="${-M_PI/2} 0.0 ${-M_PI/2}" />
-						<parent link="zed_camera_depth_frame" />
-						<child link="zed_camera_depth_optical_frame"/>
-				</joint>
-				<link name="zed_camera_depth_optical_frame"/>
-				<joint name="zed_camera_rgb_joint" type="fixed">
-						<origin xyz="0.0 -0.0125 0.0" rpy="0 0 0" />
-						<parent link="bow/camera_link" />
-						<child link="zed_camera_rgb_frame"/>
-				</joint>
-				<link name="zed_camera_rgb_frame"/>
-				<joint name="zed_camera_rgb_optical_joint" type="fixed">
-						<origin xyz="0 0 0" rpy="${-M_PI/2} 0.0 ${-M_PI/2}" />
-						<parent link="zed_camera_rgb_frame" />
-						<child link="zed_camera_rgb_optical_frame"/>
-				</joint>
-				<link name="zed_camera_rgb_optical_frame"/>
-		</xacro:if>
-		<!-- Set up sonar linkage and configuration >
-	<xacro:if value="$(arg sonar_enabled)" >
-		<joint name="base_link_sonar_link_joint" type="fixed">
-			<origin xyz="0 0 -0.05" rpy="0 ${M_PI/2} 0" />
-			<parent link="base_link"/>
-			<child link="sonar_link" />
-		</joint>
-		<link name="sonar_link">
-			<inertial>
-				<mass value="1"/>
-				<origin xyz="0 0 0"/>
-				<inertia ixx="0.1" ixy="0.0" ixz="0.0" iyy="0.1" iyz="0.0" izz="0.1"/>
-			</inertial>
-			<visual>
-				<origin xyz="0 0 0" rpy="0 0 0" />
-				<geometry>
-					<mesh filename="package://hector_sensors_description/meshes/sonar_sensor/max_sonar_ez4.dae"/>
-				</geometry>
-			</visual>
-			<collision>
-				<origin xyz="0 0 0" rpy="0 0 0" />
-				<geometry>
-					<box size="0.02 0.02 0.02" />
-				</geometry>
-			</collision>
-		</link>
-	</xacro:if -->
-	<!-- Hokuyo Laser -->
-	<xacro:if value="$(arg lidar_enabled)">
-			<joint name="hokuyo_joint" type="fixed">
-					<origin xyz="${shelf_length/2} 0 0.4" rpy="0 0 0"/>
-					<parent link="shelf_link"/>
-					<child link="hokuyo_link"/>
-			</joint>
-			<link name="hokuyo_link">
-					<collision>
-							<origin xyz="0 0 -0.0115" rpy="0 0 0"/>
-							<geometry>
-									<box size="0.058 0.058 0.087"/>
-							</geometry>
-					</collision>
-					<visual>
-							<origin xyz="0 0 0" rpy="0 0 0"/>
-							<geometry>
-									<mesh filename="package://hector_sensors_description/meshes/hokuyo_utm30lx/hokuyo_utm_30lx.dae"/>
-							</geometry>
-					</visual>
-					<inertial>
-							<mass value="0.27" />
-							<origin xyz="0 0 0" rpy="0 0 0"/>
-							<inertia ixx="2.632e-4" ixy="0" ixz="0" iyy="2.632e-4" iyz="0" izz="1.62e-4" />
-					</inertial>
-			</link>
-	</xacro:if>
-</robot>
+    <xacro:property name="M_PI" value="3.1415926535897931" />
+    <xacro:property name="shelf_length" value="1.85" />
+    <xacro:property name="shelf_width" value="1.01" />
+    <xacro:property name="shelf_thickness" value="0.1" />
+    <xacro:property name="camera_height" value="0.1" />
+    <!-- camera array joint -->
+    <xacro:macro name="spot_camera" params="position1 x y z yaw">
+        <joint name="${position1}_camera_joint" type="fixed">
+            <origin xyz="${x} ${y} ${z}" rpy="0 0 ${yaw}" />
+            <parent link="shelf_link"/>
+            <child link="${position1}/camera_link"/>
+        </joint>
+        <link name="${position1}/camera_link">
+            <visual>
+                <origin xyz="0 0 0" rpy="0 0 0" />
+                <geometry>
+                    <mesh filename="package://hector_sensors_description/meshes/thermaleye_camera/thermaleye_camera_hector_v2.dae" />
+                </geometry>
+            </visual>
+            <collision>
+                <origin xyz="0 0 0" rpy="0 0 0" />
+                <geometry>
+                    <mesh filename="package://hector_sensors_description/meshes/thermaleye_camera/thermaleye_camera_hector_v2.stl"/>
+                </geometry>
+            </collision>
+        </link>
+    </xacro:macro>
+    <xacro:macro name="underwater_camera" params="position1 x y z roll yaw">
+        <joint name="${position1}_camera_joint" type="fixed">
+            <origin xyz="${x} ${y} ${z}" rpy="0 ${roll} ${yaw}" />
+            <parent link="shelf_link"/>
+            <child link="${position1}/camera_link"/>
+        </joint>
+        <link name="${position1}/camera_link">
+            <visual>
+                <origin xyz="0 0 0" rpy="0 0 0" />
+                <geometry>
+                    <mesh filename="package://hector_sensors_description/meshes/thermaleye_camera/thermaleye_camera_hector_v2.dae"/>
+                </geometry>
+            </visual>
+            <collision>
+                <origin xyz="0 0 0" rpy="0 0 0" />
+                <geometry>
+                    <mesh filename="package://hector_sensors_description/meshes/thermaleye_camera/thermaleye_camera_hector_v2.stl"/>
+                </geometry>
+            </collision>
+        </link>
+    </xacro:macro>
+    <xacro:macro name="stereo_camera" params="position1 position2 x y z roll yaw">
+        <joint name="${position1}_${position2}_camera_joint" type="fixed">
+            <origin xyz="${x} ${y} ${z}" rpy="0 ${roll} ${yaw}" />
+            <parent link="shelf_link"/>
+            <child link="${position1}/${position2}/camera_link"/>
+        </joint>
+        <link name="${position1}/${position2}/camera_link">
+            <visual>
+                <origin xyz="0 0 0" rpy="0 0 0" />
+                <geometry>
+                    <mesh filename="package://hector_sensors_description/meshes/thermaleye_camera/thermaleye_camera_hector_v2.dae"/>
+                </geometry>
+            </visual>
+            <collision>
+                <origin xyz="0 0 0" rpy="0 0 0" />
+                <geometry>
+                    <mesh filename="package://hector_sensors_description/meshes/thermaleye_camera/thermaleye_camera_hector_v2.stl"/>
+                </geometry>
+            </collision>
+        </link>
+    </xacro:macro>
+    <joint name="gps_joint" type="fixed">
+        <origin xyz="0 0 ${shelf_thickness*6}" rpy="0 0 0" />
+        <parent link="shelf_link"/>
+        <child link="gps_link"/>
+    </joint>
+    <link name="gps_link">
+        <visual>
+            <origin xyz="0 0 0" rpy="0 0 0"/>
+            <geometry>
+                <cylinder length="0.08" radius="0.1" />
+            </geometry>
+            <material name="white" />
+        </visual>
+        <collision>
+            <origin xyz="0 0 0" rpy="0 0 0"/>
+            <geometry>
+                <cylinder length="0.08" radius="0.1" />
+            </geometry>
+        </collision>
+    </link>
+    <xacro:unless value="$(arg zed_enabled)" >
+        <xacro:stereo_camera position1="bow" position2="left" x="${shelf_length/2+0.2}" y="${shelf_width/4}" z="${camera_height}" roll="0.157" yaw="0"/>
+        <xacro:stereo_camera position1="bow" position2="right" x="${shelf_length/2+0.2}" y="-${shelf_width/4}" z="${camera_height}" roll="0.157" yaw="0"/>
+    </xacro:unless>
+    <xacro:underwater_camera position1="underwater" x="${shelf_length/2}" y="${shelf_width/2}" z="-1" roll="${PI/2}" yaw="0"/>
+    <xacro:spot_camera position1="port" x="${shelf_length/2}" y="${shelf_width/2}" z="${camera_height}" yaw="${PI/2}"/>
+    <xacro:spot_camera position1="starboard" x="${shelf_length/2}" y="-${shelf_width/2}" z="${camera_height}" yaw="-${PI/2}"/>
+    <xacro:spot_camera position1="transom" x="-${1.8*shelf_width/2}" y="0" z="${camera_height}" yaw="${PI}"/>
+    <!--zed camera -->
+    <xacro:if value="$(arg zed_enabled)" >
+        <joint name="zed_camera_joint" type="fixed">
+            <origin xyz="${shelf_length/2+0.2} 0 ${camera_height}" rpy="0 0 0" />
+            <parent link="shelf_link"/>
+            <child link="bow/camera_link"/>
+        </joint>
+        <link name="bow/camera_link">
+            <inertial>
+                <mass value="0.01" />
+                <origin xyz="0 0 0" rpy="0 0 0"/>
+                <inertia ixx="2.632e-4" ixy="0" ixz="0" iyy="2.632e-4" iyz="0" izz="1.62e-4" />
+            </inertial>
+            <!--visual>
+                <origin xyz="0 0 0" rpy="${PI/2} 0 ${PI/2}" />
+                <geometry>
+                    <mesh filename="package://robotx_description/meshes/zed_model.dae" scale="0.05 0.05 0.05"/>
+                </geometry>
+            </visual>
+            <collision>
+                <origin xyz="0 0 0" rpy="${PI/2} 0 ${PI/2}" />
+                <geometry>
+                    <mesh filename="package://robotx_description/meshes/zed_model.dae" scale="0.05 0.05 0.05"/>
+                </geometry>
+            </collision-->
+            <inertial>
+                <mass value="0.01" />
+                <origin xyz="0 0 0" rpy="0 0 0"/>
+                <inertia ixx="2.632e-4" ixy="0" ixz="0" iyy="2.632e-4" iyz="0" izz="1.62e-4" />
+            </inertial>
+            <visual>
+                <origin xyz="0 0 0" rpy="0 0 0" />
+                <geometry>
+                    <mesh filename="package://hector_sensors_description/meshes/kinect_camera/kinect_camera_simple.dae"/>
+                </geometry>
+            </visual>
+            <collision>
+                <origin xyz="0 0 0" rpy="0 0 0" />
+                <geometry>
+                    <mesh filename="package://hector_sensors_description/meshes/kinect_camera/kinect_camera_simple.stl"/>
+                </geometry>
+            </collision>
+        </link>
+        <joint name="zed_camera_depth_joint" type="fixed">
+            <origin xyz="0.0 -0.01 0.0" rpy="0 0 0" />
+            <parent link="bow/camera_link" />
+            <child link="bow/camera_depth_frame"/>
+        </joint>
+        <link name="bow/camera_depth_frame"/>
+        <joint name="zed_camera_depth_optical_joint" type="fixed">
+            <origin xyz="0 0 0" rpy="${-M_PI/2} 0.0 ${-M_PI/2}" />
+            <parent link="bow/camera_depth_frame" />
+            <child link="bow/camera_depth_optical_frame"/>
+        </joint>
+        <link name="bow/camera_depth_optical_frame"/>
+        <joint name="zed_camera_rgb_joint" type="fixed">
+            <origin xyz="0.0 -0.0125 0.0" rpy="0 0 0" />
+            <parent link="bow/camera_link" />
+            <child link="bow/camera_rgb_frame"/>
+        </joint>
+        <link name="bow/camera_rgb_frame"/>
+        <joint name="zed_camera_rgb_optical_joint" type="fixed">
+            <origin xyz="0 0 0" rpy="${-M_PI/2} 0.0 ${-M_PI/2}" />
+            <parent link="bow/camera_rgb_frame" />
+            <child link="bow/camera_rgb_optical_frame"/>
+        </joint>
+        <link name="bow/camera_rgb_optical_frame"/>
+    </xacro:if>
+    <!-- Set up sonar linkage and configuration >
+        <xacro:if value="$(arg sonar_enabled)" >
+                <joint name="base_link_sonar_link_joint" type="fixed">
+                        <origin xyz="0 0 -0.05" rpy="0 ${M_PI/2} 0" />
+                        <parent link="base_link"/>
+                        <child link="sonar_link" />
+                </joint>
+                <link name="sonar_link">
+                        <inertial>
+                                <mass value="1"/>
+                                <origin xyz="0 0 0"/>
+                                <inertia ixx="0.1" ixy="0.0" ixz="0.0" iyy="0.1" iyz="0.0" izz="0.1"/>
+                        </inertial>
+                        <visual>
+                                <origin xyz="0 0 0" rpy="0 0 0" />
+                                <geometry>
+                                        <mesh filename="package://hector_sensors_description/meshes/sonar_sensor/max_sonar_ez4.dae"/>
+                                </geometry>
+                        </visual>
+                        <collision>
+                                <origin xyz="0 0 0" rpy="0 0 0" />
+                                <geometry>
+                                        <box size="0.02 0.02 0.02" />
+                                </geometry>
+                        </collision>
+                </link>
+        </xacro:if -->
+        <!-- Hokuyo Laser -->
+        <xacro:if value="$(arg lidar_enabled)">
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